Commit message: Adjust and check static robot visualization

File: description/camera.xacro (robot description, xacro)
@@ -1,2 +1,3 @@
+<robot xmlns:xacro="http://www.ros.org/wiki/xacro">
     <joint name="camera_joint" type="fixed">
         <parent link="chassis"/>
@@ -48,2 +49,3 @@
         </sensor>
     </gazebo>
+</robot>

File: description/common_platform.urdf.xacro (robot description, xacro)
@@ -11,5 +11,5 @@
     </xacro:unless>
     <xacro:include filename="lidar.xacro" />
-    <xacro:include filename="camera.xacro" />
+    <!-- <xacro:include filename="camera.xacro" /> -->
     <!-- <xacro:include filename="depth_camera.xacro" /> -->
     <!-- <xacro:include filename="face.xacro" /> -->

File: description/inertial_macros.xacro (robot description, xacro)
@@ -1,2 +1,3 @@
+<robot xmlns:xacro="http://www.ros.org/wiki/xacro">
     <!-- Specify some standard inertial calculations https://en.wikipedia.org/wiki/List_of_moments_of_inertia -->
     <!-- These make use of xacro's mathematical functionality -->
@@ -28,2 +29,3 @@
         </inertial>
     </xacro:macro>
+</robot>

File: description/lidar.xacro (robot description, xacro)
@@ -1,28 +1,24 @@
+<robot xmlns:xacro="http://www.ros.org/wiki/xacro">
     <joint name="laser_joint" type="fixed">
         <parent link="chassis"/>
         <child link="laser_frame"/>
-        <origin xyz="0.122 0 0.212" rpy="0 0 0"/>
+        <origin xyz="-0.032146 0.0017 .12155" rpy="0 0 -1.5708"/>
     </joint>
     <link name="laser_frame">
         <visual>
+            <origin xyz="0 0 -0.04525"/>
             <geometry>
-                <cylinder radius="0.05" length="0.04"/>
-            </geometry>
-            <material name="black"/>
-        </visual>
-        <visual>
-            <origin xyz="0 0 -0.05"/>
-            <geometry>
-                <cylinder radius="0.01" length="0.1"/>
+                <mesh filename="package://common_platform/meshes/RPLidarA1M8Kit.stl" scale=".001 .001 .001"/>
             </geometry>
             <material name="black"/>
         </visual>
         <collision>
+            <origin xyz="0 0 -0.0235" rpy="0 0 0"/>
             <geometry>
-                <cylinder radius="0.05" length="0.04"/>
+                <cylinder radius="0.065" length="0.055"/>
             </geometry>
         </collision>
-        <xacro:inertial_cylinder mass="0.1" length="0.04" radius="0.05">
-            <origin xyz="0 0 0" rpy="0 0 0"/>
+        <xacro:inertial_cylinder mass="0.17" length="0.055" radius="0.065">
+            <origin xyz="0 0 -0.0235" rpy="0 0 0"/>
         </xacro:inertial_cylinder>
     </link>
@@ -42,5 +38,5 @@
                 </scan>
                 <range>
-                    <min>0.3</min>
+                    <min>0.15</min>
                     <max>12</max>
                 </range>
@@ -55,2 +51,3 @@
         </sensor>
     </gazebo>
+</robot>

File: description/robot_core.xacro (robot description, xacro)
@@ -1,17 +1,17 @@
 <?xml version="1.0"?>
+<robot xmlns:xacro="http://www.ros.org/wiki/xacro">
     <xacro:include filename="inertial_macros.xacro"/>
-    <xacro:property name="chassis_length" value="0.335"/>
-    <xacro:property name="chassis_width" value="0.265"/>
-    <xacro:property name="chassis_height" value="0.138"/>
+    <xacro:property name="chassis_diameter" value="0.245"/>
+    <xacro:property name="chassis_height" value="0.1013"/>
     <xacro:property name="chassis_mass" value="1.0"/>
-    <xacro:property name="wheel_radius" value="0.033"/>
-    <xacro:property name="wheel_thickness" value="0.026"/>
+    <xacro:property name="wheel_radius" value="0.035"/>
+    <xacro:property name="wheel_thickness" value="0.008"/>
     <xacro:property name="wheel_mass" value="0.05"/>
-    <xacro:property name="wheel_offset_x" value="0.226"/>
-    <xacro:property name="wheel_offset_y" value="0.1485"/>
-    <xacro:property name="wheel_offset_z" value="0.01"/>
-    <xacro:property name="caster_wheel_radius" value="0.01"/>
+    <xacro:property name="wheel_offset_x" value="0.000"/>
+    <xacro:property name="wheel_offset_y" value="0.07039"/>
+    <xacro:property name="wheel_offset_z" value="0.010"/>
+    <xacro:property name="caster_wheel_radius" value="0.013"/>
     <xacro:property name="caster_wheel_mass" value="0.01"/>
-    <xacro:property name="caster_wheel_offset_x" value="0.075"/>
+    <xacro:property name="caster_wheel_offset_x" value="0.044174"/>
     <xacro:property name="caster_wheel_offset_z" value="${wheel_offset_z - wheel_radius + caster_wheel_radius}"/>
     <material name="white">
@@ -37,5 +37,5 @@
         <parent link="base_link"/>
         <child link="base_footprint"/>
-        <origin xyz="0 0 0" rpy="0 0 0"/>
+        <origin xyz="0 0 ${-wheel_radius}" rpy="0 0 0"/>
     </joint>
     <link name="base_footprint">
@@ -49,19 +49,19 @@
     <link name="chassis">
         <visual>
-            <origin xyz="${chassis_length/2} 0 ${chassis_height/2}"/>
+            <origin xyz="0 0 0" rpy="0 0 0"/>
             <geometry>
-                <box size="${chassis_length} ${chassis_width} ${chassis_height}"/>
+                <mesh filename="package://common_platform/meshes/chassis.stl" scale=".001 .001 .001"/>
             </geometry>
             <material name="orange"/>
         </visual>
         <collision>
-            <origin xyz="${chassis_length/2} 0 ${chassis_height/2}"/>
+            <origin xyz="${chassis_diameter/2} 0 ${wheel_offset_z - wheel_radius + chassis_height/2}"/>
             <geometry>
-                <box size="${chassis_length} ${chassis_width} ${chassis_height}"/>
+                <cylinder radius="${chassis_diameter/2}" length="${chassis_height}"/>
             </geometry>
         </collision>
-        <xacro:inertial_box mass="0.5" x="${chassis_length}" y="${chassis_width}" z="${chassis_height}">
-            <origin xyz="${chassis_length/2} 0 ${chassis_height/2}" rpy="0 0 0"/>
-        </xacro:inertial_box>
+        <xacro:inertial_cylinder mass="0.5" length="${chassis_height}" radius="${chassis_diameter/2}">
+            <origin xyz="0 0 ${wheel_offset_z - wheel_radius + chassis_height/2}" rpy="0 0 0"/>
+        </xacro:inertial_cylinder>
     </link>
     <gazebo reference="chassis">
@@ -147,2 +147,3 @@
         <mu2 value="0.001"/>
     </gazebo>
+</robot>

File: description/ros2_control.xacro (robot description, xacro)
@@ -1,2 +1,3 @@
+<robot xmlns:xacro="http://www.ros.org/wiki/xacro">
     <xacro:unless value="$(arg sim_mode)">
         <ros2_control name="RealRobot" type="system">
@@ -58,2 +59,3 @@
         </plugin>
     </gazebo>
+</robot>
